Commit message: Fix UR10 hybrid planner demo runtime

File: ipa_moveit_config/srdf/ur_macro.srdf.xacro (robot description, xacro)
@@ -41,5 +41,5 @@
     <!--END EFFECTOR - Purpose - Represent information about an end effector.-->
     <!--VIRTUAL JOINT - Purpose - this element defines a virtual joint between a robot link and an external frame of reference (considered fixed with respect to the robot)-->
-    <virtual_joint name="${prefix}fixed_base" type="fixed" parent_frame="world" child_link="${prefix}base_link" />
+    <joint name="${prefix}fixed_base" type="fixed" parent_frame="world" child_link="${prefix}base_link" />
     <!--DISABLE COLLISIONS - By default it is assumed that any link of the robot could potentially come into collision with any other link in the robot. This tag disables collision checking between a specified pair of links. -->
     <disable_collisions link1="${prefix}base_link" link2="${prefix}base_link_inertia" reason="Adjacent" />

Commit message: Set joint state and cartesian plan that is good for welding demo

File: ipa_moveit_config/srdf/ur_macro.srdf.xacro (robot description, xacro)
@@ -39,4 +39,12 @@
       <joint name="${prefix}wrist_3_joint" value="-0.11" />
     </group_state>
+    <group_state name="${prefix}pre_welding_configuration" group="${prefix}${name}_manipulator">
+      <joint name="${prefix}elbow_joint" value="1.744" />
+      <joint name="${prefix}shoulder_lift_joint" value="-1.506" />
+      <joint name="${prefix}shoulder_pan_joint" value="0.838" />
+      <joint name="${prefix}wrist_1_joint" value="-1.712" />
+      <joint name="${prefix}wrist_2_joint" value="-1.691" />
+      <joint name="${prefix}wrist_3_joint" value="-0.809" />
+    </group_state>
     <!--END EFFECTOR - Purpose - Represent information about an end effector.-->
     <!--VIRTUAL JOINT - Purpose - this element defines a virtual joint between a robot link and an external frame of reference (considered fixed with respect to the robot)-->

Commit message: Update calibration, cartesian limits and add welding tip required by MTC

File: ipa_moveit_config/srdf/ur_macro.srdf.xacro (robot description, xacro)
@@ -13,4 +13,7 @@
     <group name="${prefix}${name}_manipulator">
       <chain base_link="${prefix}base_link" tip_link="tcp_welding_gun_link" />
+    </group>
+    <group name="welding_gun">
+        <link name="tcp_welding_gun_link" />
     </group>
     <!--GROUP STATES - Purpose - Define a named state for a particular group, in terms of joint values. This is useful to define states like 'folded arms'-->
@@ -48,4 +51,5 @@
     </group_state>
     <!--END EFFECTOR - Purpose - Represent information about an end effector.-->
+    <end_effector name="welding_ee" parent_link="tcp_welding_gun_link" group="welding_gun" />
     <!--VIRTUAL JOINT - Purpose - this element defines a virtual joint between a robot link and an external frame of reference (considered fixed with respect to the robot)-->
     <joint name="${prefix}fixed_base" type="fixed" parent_frame="world" child_link="${prefix}base_link" />
