Commit message: ipa_ur_demo.urdf.xacro: Remove walls for fake hardware

File: ipa_demo_cell_description/urdf/ipa_demo_env.urdf.xacro (robot description, xacro)
@@ -4,5 +4,5 @@
      For more information, please see http://wiki.ros.org/sw_urdf_exporter -->
 <robot xmlns:xacro="http://wiki.ros.org/xacro">
-  <xacro:macro name="ipa_demo_env" params="prefix">
+  <xacro:macro name="ipa_demo_env" params="prefix use_fake_hardware:=false">
     <link name="env_link">
       <inertial>
@@ -28,54 +28,47 @@
     </link>
     <!-- Add boxes for collision detection -->
-    <joint name="left_box" type="fixed">
-      <parent link="env_link" />
-      <child link="left_box" />
-      <origin xyz="0 1.5 -1.05" rpy="0 0 0" />
-    </joint>
-    <joint name="right_box" type="fixed">
-      <parent link="env_link" />
-      <child link="right_box" />
-      <origin xyz="0 1.5 1.05" rpy="0 0 0" />
-    </joint>
-    <joint name="back_box" type="fixed">
-      <parent link="env_link" />
-      <child link="back_box" />
-      <origin xyz="-1.4 1.5 0" rpy="0 0 0" />
-    </joint>
-    <!-- <joint name="front_box" type="fixed">
+    <xacro:unless value="${use_fake_hardware}">
+      <joint name="left_box" type="fixed">
         <parent link="env_link" />
-        <child link="front_box" />
-        <origin xyz="1.45 1.5 0" rpy="0 0 0" />
-      </joint> -->
-    <joint name="top_box" type="fixed">
-      <parent link="env_link" />
-      <child link="top_box" />
-      <origin xyz="0 2.35 0 " rpy="0 0 0" />
-    </joint>
-    <link name="left_box">
-      <collision>
-        <origin xyz="0 0 0" rpy="0 0 0"/>
-        <geometry>
-          <box size="3.0 3.0 0.1"/>
-        </geometry>
-      </collision>
-    </link>
-    <link name="right_box">
-      <collision>
-        <origin xyz="0 0 0" rpy="0 0 0"/>
-        <geometry>
-          <box size="3.0 3.0 0.1"/>
-        </geometry>
-      </collision>
-    </link>
-    <link name="back_box">
-      <collision>
-        <origin xyz="0 0 0" rpy="0 0 0"/>
-        <geometry>
-          <box size="0.1 3.0 3.0"/>
-        </geometry>
-      </collision>
-    </link>
-    <!-- <link name="front_box">
+        <child link="left_box" />
+        <origin xyz="0 1.5 -1.05" rpy="0 0 0" />
+      </joint>
+      <joint name="right_box" type="fixed">
+        <parent link="env_link" />
+        <child link="right_box" />
+        <origin xyz="0 1.5 1.05" rpy="0 0 0" />
+      </joint>
+      <joint name="back_box" type="fixed">
+        <parent link="env_link" />
+        <child link="back_box" />
+        <origin xyz="-1.4 1.5 0" rpy="0 0 0" />
+      </joint>
+      <!-- <joint name="front_box" type="fixed">
+          <parent link="env_link" />
+          <child link="front_box" />
+          <origin xyz="1.45 1.5 0" rpy="0 0 0" />
+        </joint> -->
+      <joint name="top_box" type="fixed">
+        <parent link="env_link" />
+        <child link="top_box" />
+        <origin xyz="0 2.35 0 " rpy="0 0 0" />
+      </joint>
+      <link name="left_box">
+        <collision>
+          <origin xyz="0 0 0" rpy="0 0 0"/>
+          <geometry>
+            <box size="3.0 3.0 0.1"/>
+          </geometry>
+        </collision>
+      </link>
+      <link name="right_box">
+        <collision>
+          <origin xyz="0 0 0" rpy="0 0 0"/>
+          <geometry>
+            <box size="3.0 3.0 0.1"/>
+          </geometry>
+        </collision>
+      </link>
+      <link name="back_box">
         <collision>
           <origin xyz="0 0 0" rpy="0 0 0"/>
@@ -84,13 +77,22 @@
           </geometry>
         </collision>
-      </link> -->
-    <link name="top_box">
-      <collision>
-        <origin xyz="0 0 0" rpy="0 0 0"/>
-        <geometry>
-          <box size="3.0 0.1 3.0"/>
-        </geometry>
-      </collision>
-    </link>
+      </link>
+      <!-- <link name="front_box">
+          <collision>
+            <origin xyz="0 0 0" rpy="0 0 0"/>
+            <geometry>
+              <box size="0.1 3.0 3.0"/>
+            </geometry>
+          </collision>
+        </link> -->
+      <link name="top_box">
+        <collision>
+          <origin xyz="0 0 0" rpy="0 0 0"/>
+          <geometry>
+            <box size="3.0 0.1 3.0"/>
+          </geometry>
+        </collision>
+      </link>
+    </xacro:unless>
   </xacro:macro>
 </robot>

File: ipa_demo_cell_description/urdf/ipa_ur_demo.urdf.xacro (robot description, xacro)
@@ -40,5 +40,7 @@
   <xacro:include filename="$(find ipa_demo_cell_description)/urdf/ipa_demo_env.urdf.xacro" />
   <link name="world" />
-  <xacro:ipa_demo_env prefix="" />
+  <xacro:ipa_demo_env
+    prefix=""
+    use_fake_hardware="$(arg use_fake_hardware)" />
   <joint name="demo_env_joint" type="fixed">
     <parent link="world" />

Commit message: Update robot layout and calibration

File: ipa_demo_cell_description/urdf/ipa_demo_env.urdf.xacro (robot description, xacro)
@@ -4,10 +4,10 @@
      For more information, please see http://wiki.ros.org/sw_urdf_exporter -->
 <robot xmlns:xacro="http://wiki.ros.org/xacro">
-  <xacro:macro name="ipa_demo_env" params="prefix use_fake_hardware:=false">
+  <xacro:macro name="ipa_demo_env" params="prefix">
     <link name="env_link">
       <inertial>
-        <origin xyz="-0.0741666676689185 0.587693158719805 -8.80953956550394E-16" rpy="0 0 0" />
-        <mass value="16.4612070211758" />
-        <inertia ixx="2.52303308496007" ixy="-4.63618882129208E-16" ixz="-1.63654706343414E-15" iyy="3.85345752503351" iyz="1.5738466691302E-15" izz="2.52303308496007" />
+        <origin xyz="-0.0710821713973007 1.04952300655296E-15 0.586534037453751" rpy="0 0 0" />
+        <mass value="16.2791658374424" />
+        <inertia ixx="2.50656922244652" ixy="-1.54202348047649E-15" ixz="9.02523734700172E-16" iyy="2.50656922244652" iyz="-8.39298741609604E-16" izz="3.81563122590028" />
       </inertial>
       <visual>
@@ -28,71 +28,69 @@
     </link>
     <!-- Add boxes for collision detection -->
-    <xacro:unless value="${use_fake_hardware}">
-      <joint name="left_box" type="fixed">
-        <parent link="env_link" />
-        <child link="left_box" />
-        <origin xyz="0 1.5 -1.05" rpy="0 0 0" />
-      </joint>
-      <joint name="right_box" type="fixed">
-        <parent link="env_link" />
-        <child link="right_box" />
-        <origin xyz="0 1.5 1.05" rpy="0 0 0" />
-      </joint>
-      <joint name="back_box" type="fixed">
-        <parent link="env_link" />
-        <child link="back_box" />
-        <origin xyz="-1.4 1.5 0" rpy="0 0 0" />
-      </joint>
-      <!-- <joint name="front_box" type="fixed">
-          <parent link="env_link" />
-          <child link="front_box" />
-          <origin xyz="1.45 1.5 0" rpy="0 0 0" />
-        </joint> -->
-      <joint name="top_box" type="fixed">
-        <parent link="env_link" />
-        <child link="top_box" />
-        <origin xyz="0 2.35 0 " rpy="0 0 0" />
-      </joint>
-      <link name="left_box">
-        <collision>
-          <origin xyz="0 0 0" rpy="0 0 0"/>
-          <geometry>
-            <box size="3.0 3.0 0.1"/>
-          </geometry>
-        </collision>
-      </link>
-      <link name="right_box">
-        <collision>
-          <origin xyz="0 0 0" rpy="0 0 0"/>
-          <geometry>
-            <box size="3.0 3.0 0.1"/>
-          </geometry>
-        </collision>
-      </link>
-      <link name="back_box">
-        <collision>
-          <origin xyz="0 0 0" rpy="0 0 0"/>
-          <geometry>
-            <box size="0.1 3.0 3.0"/>
-          </geometry>
-        </collision>
-      </link>
-      <!-- <link name="front_box">
-          <collision>
-            <origin xyz="0 0 0" rpy="0 0 0"/>
-            <geometry>
-              <box size="0.1 3.0 3.0"/>
-            </geometry>
-          </collision>
-        </link> -->
-      <link name="top_box">
-        <collision>
-          <origin xyz="0 0 0" rpy="0 0 0"/>
-          <geometry>
-            <box size="3.0 0.1 3.0"/>
-          </geometry>
-        </collision>
-      </link>
-    </xacro:unless>
+    <joint name="left_box" type="fixed">
+      <parent link="env_link" />
+      <child link="left_box" />
+      <origin xyz="0 1.0 1.25" rpy="0 0 0" />
+    </joint>
+    <joint name="right_box" type="fixed">
+      <parent link="env_link" />
+      <child link="right_box" />
+      <origin xyz="0 -1.0 1.25" rpy="0 0 0" />
+    </joint>
+    <joint name="back_box" type="fixed">
+      <parent link="env_link" />
+      <child link="back_box" />
+      <origin xyz="-1.4 0 1.25" rpy="0 0 0" />
+    </joint>
+    <joint name="front_box" type="fixed">
+      <parent link="env_link" />
+      <child link="front_box" />
+      <origin xyz="1.4 0 1.25" rpy="0 0 0" />
+    </joint>
+    <joint name="top_box" type="fixed">
+      <parent link="env_link" />
+      <child link="top_box" />
+      <origin xyz="0 0 2.5 " rpy="0 0 0" />
+    </joint>
+    <link name="left_box">
+      <collision>
+        <origin xyz="0 0 0" rpy="0 0 0"/>
+        <geometry>
+          <box size="3.0 0.1 2.5 "/>
+        </geometry>
+      </collision>
+    </link>
+    <link name="right_box">
+      <collision>
+        <origin xyz="0 0 0" rpy="0 0 0"/>
+        <geometry>
+          <box size="3.0 0.1 2.5 "/>
+        </geometry>
+      </collision>
+    </link>
+    <link name="back_box">
+      <collision>
+        <origin xyz="0 0 0" rpy="0 0 0"/>
+        <geometry>
+          <box size="0.1 3.0 2.5"/>
+        </geometry>
+      </collision>
+    </link>
+    <link name="front_box">
+      <collision>
+        <origin xyz="0 0 0" rpy="0 0 0"/>
+        <geometry>
+          <box size="0.1 3.0 2.5"/>
+        </geometry>
+      </collision>
+    </link>
+    <link name="top_box">
+      <collision>
+        <origin xyz="0 0 0" rpy="0 0 0"/>
+        <geometry>
+          <box size="3.0 3.0 0.1"/>
+        </geometry>
+      </collision>
+    </link>
   </xacro:macro>
 </robot>

File: ipa_demo_cell_description/urdf/ipa_ur_demo.urdf.xacro (robot description, xacro)
@@ -43,11 +43,9 @@
   <xacro:include filename="$(find ipa_demo_cell_description)/urdf/ipa_demo_env.urdf.xacro" />
   <link name="world" />
-  <xacro:ipa_demo_env
-    prefix=""
-    use_fake_hardware="$(arg use_fake_hardware)" />
+  <xacro:ipa_demo_env prefix="" />
   <joint name="demo_env_joint" type="fixed">
     <parent link="world" />
     <child link="env_link" />
-    <origin xyz="0 0 0" rpy="${pi/2} 0 0"/>
+    <origin xyz="0 0 0" rpy="0 0 0"/>
   </joint>
   <!-- Attach UR to environment -->
@@ -55,5 +53,5 @@
     <parent link="env_link" />
     <child link="base_link" />
-    <origin xyz="-0.350 0.766 0" rpy="-${pi/2} -${pi/2} 0" />
+    <origin xyz="-0.350 0 0.813" rpy="0 0 ${-pi/2}" />
   </joint>
   <!-- Sensor calibration -->

File: ipa_demo_cell_description/urdf/welding_gun_lorch_scancontrol_3000.urdf.xacro (robot description, xacro)
@@ -7,7 +7,7 @@
     <link name="welding_gun_link">
       <inertial>
-        <origin xyz="-0.0785750635579513 0.0478255317464427 -0.281129549529667" rpy="0 0 0" />
-        <mass value="1.86859564603062" />
-        <inertia ixx="0.00485321168704067" ixy="-8.98634828494543E-05" ixz="-0.00150096446074707" iyy="0.00978317996859146" iyz="-0.000164554654502753" izz="0.00695496569317101" />
+        <origin xyz="-0.063966723890025 0.0507342971013102 -0.279018970359549" rpy="0 0 0" />
+        <mass value="1.76093615205291" />
+        <inertia ixx="0.0048143448063882" ixy="-8.94621372608532E-05" ixz="-0.00151145048825125" iyy="0.0097571665662651" iyz="-0.000167961449930583" izz="0.00691320517040876" />
       </inertial>
       <visual>
@@ -23,5 +23,5 @@
         <origin xyz="0 0 0" rpy="0 0 0" />
         <geometry>
-          <mesh filename="package://ipa_demo_cell_description/meshes/welding_gun_lorch_scancontrol_3000.STL" />
+          <mesh filename="package://ipa_demo_cell_description/meshes/welding_gun_lorch_scancontrol_3000_collision.STL" />
         </geometry>
       </collision>
