Commit message: Change URDF for UR5e

File: ipa_demo_cell_description/urdf/ipa_ur_demo.urdf.xacro (robot description, xacro)
@@ -54,5 +54,5 @@
   <!-- Sensor calibration -->
   <!-- Set the tcp according to Hand Eye Calibration-->
-  <xacro:property name="sensor_config" value="${load_yaml('$(arg calibration_config_file)')}" />
+  <!-- <xacro:property name="sensor_config" value="${load_yaml('$(arg calibration_config_file)')}" />
   <xacro:property name="tcp_sensor" value="${sensor_config['tcp_sensor']}"/>
   <link name="tcp_sensor_link" />
@@ -65,7 +65,7 @@
                  ${tcp_sensor['pitch']}
                  ${tcp_sensor['yaw']}"/>
-  </joint>
+  </joint> -->
   <!-- Set the welding gun tool-->
-  <xacro:property name="welding_gun_config" value="${load_yaml('$(arg calibration_config_file)')}" />
+  <!-- <xacro:property name="welding_gun_config" value="${load_yaml('$(arg calibration_config_file)')}" />
   <xacro:property name="tcp_welding_gun" value="${welding_gun_config['tcp_welding_gun']}"/>
   <link name="tcp_welding_gun_link" />
@@ -78,7 +78,7 @@
                  ${tcp_welding_gun['pitch']}
                  ${tcp_welding_gun['yaw']}"/>
-  </joint>
+  </joint> -->
   <!-- Attach the welding gun -->
-  <xacro:include filename="$(find ipa_demo_cell_description)/urdf/$(arg endeffector).urdf.xacro" />
+  <!-- <xacro:include filename="$(find ipa_demo_cell_description)/urdf/$(arg endeffector).urdf.xacro" />
   <xacro:endeffector prefix="" />
   <xacro:property name="flange_welding_gun" value="${welding_gun_config['flange_welding_gun']}"/>
@@ -91,4 +91,26 @@
                  ${flange_welding_gun['pitch']}
                  ${flange_welding_gun['yaw']}"/>
+  </joint> -->
+  <link name="tcp_welding_gun_link" >
+    <visual>
+      <origin xyz="0 0 -0.07" rpy="0 0 0" />
+      <geometry>
+        <cylinder radius="0.01" length="0.14"/>
+      </geometry>
+      <material name="Cyan">
+        <color rgba="0 1.0 1.0 1.0"/>
+      </material>
+    </visual>
+    <collision>
+      <origin xyz="0 0 0.07" rpy="0 0 0"/>
+      <geometry>
+        <cylinder radius="0.01" length="0.14"/>
+      </geometry>
+    </collision>
+  </link>
+  <joint name="tcp_welding_gun_joint" type="fixed">
+    <parent link="wrist_3_link"/>
+    <child link="tcp_welding_gun_link"/>
+    <origin xyz="0 0 0.14" rpy="0 0 0"/>
   </joint>
 </robot>

File: ipa_moveit_config/srdf/ur_macro.srdf.xacro (robot description, xacro)
@@ -54,4 +54,6 @@
     <disable_collisions link1="${prefix}wrist_1_link" link2="${prefix}wrist_3_link" reason="Never" />
     <disable_collisions link1="${prefix}wrist_2_link" link2="${prefix}wrist_3_link" reason="Adjacent" />
+    <disable_collisions link1="welding_gun_link" link2="${prefix}wrist_3_link" reason="Adjacent" />
+    <disable_collisions link1="base_link_inertia" link2="env_link" reason="Adjacent" />
   </xacro:macro>
 </robot>

Commit message: Change fake weld link to box so you can see it rotate

File: ipa_demo_cell_description/urdf/ipa_ur_demo.urdf.xacro (robot description, xacro)
@@ -96,5 +96,6 @@
       <origin xyz="0 0 -0.07" rpy="0 0 0" />
       <geometry>
-        <cylinder radius="0.01" length="0.14"/>
+        <box size="0.01 0.01 0.14" />
+        <!-- <cylinder radius="0.01" length="0.14"/> -->
       </geometry>
       <material name="Cyan">
@@ -105,5 +106,6 @@
       <origin xyz="0 0 0.07" rpy="0 0 0"/>
       <geometry>
-        <cylinder radius="0.01" length="0.14"/>
+        <box size="0.01 0.01 0.14" />
+        <!-- <cylinder radius="0.01" length="0.14"/> -->
       </geometry>
     </collision>

Commit message: Go back to UR10e Welding URDF

File: ipa_demo_cell_description/urdf/ipa_ur_demo.urdf.xacro (robot description, xacro)
@@ -54,5 +54,5 @@
   <!-- Sensor calibration -->
   <!-- Set the tcp according to Hand Eye Calibration-->
-  <!-- <xacro:property name="sensor_config" value="${load_yaml('$(arg calibration_config_file)')}" />
+  <xacro:property name="sensor_config" value="${load_yaml('$(arg calibration_config_file)')}" />
   <xacro:property name="tcp_sensor" value="${sensor_config['tcp_sensor']}"/>
   <link name="tcp_sensor_link" />
@@ -65,7 +65,7 @@
                  ${tcp_sensor['pitch']}
                  ${tcp_sensor['yaw']}"/>
-  </joint> -->
+  </joint>
   <!-- Set the welding gun tool-->
-  <!-- <xacro:property name="welding_gun_config" value="${load_yaml('$(arg calibration_config_file)')}" />
+  <xacro:property name="welding_gun_config" value="${load_yaml('$(arg calibration_config_file)')}" />
   <xacro:property name="tcp_welding_gun" value="${welding_gun_config['tcp_welding_gun']}"/>
   <link name="tcp_welding_gun_link" />
@@ -78,7 +78,7 @@
                  ${tcp_welding_gun['pitch']}
                  ${tcp_welding_gun['yaw']}"/>
-  </joint> -->
+  </joint>
   <!-- Attach the welding gun -->
-  <!-- <xacro:include filename="$(find ipa_demo_cell_description)/urdf/$(arg endeffector).urdf.xacro" />
+  <xacro:include filename="$(find ipa_demo_cell_description)/urdf/$(arg endeffector).urdf.xacro" />
   <xacro:endeffector prefix="" />
   <xacro:property name="flange_welding_gun" value="${welding_gun_config['flange_welding_gun']}"/>
@@ -91,28 +91,4 @@
                  ${flange_welding_gun['pitch']}
                  ${flange_welding_gun['yaw']}"/>
-  </joint> -->
-  <link name="tcp_welding_gun_link" >
-    <visual>
-      <origin xyz="0 0 -0.07" rpy="0 0 0" />
-      <geometry>
-        <box size="0.01 0.01 0.14" />
-        <!-- <cylinder radius="0.01" length="0.14"/> -->
-      </geometry>
-      <material name="Cyan">
-        <color rgba="0 1.0 1.0 1.0"/>
-      </material>
-    </visual>
-    <collision>
-      <origin xyz="0 0 0.07" rpy="0 0 0"/>
-      <geometry>
-        <box size="0.01 0.01 0.14" />
-        <!-- <cylinder radius="0.01" length="0.14"/> -->
-      </geometry>
-    </collision>
-  </link>
-  <joint name="tcp_welding_gun_joint" type="fixed">
-    <parent link="wrist_3_link"/>
-    <child link="tcp_welding_gun_link"/>
-    <origin xyz="0 0 0.14" rpy="0 0 0"/>
   </joint>
 </robot>

Commit message: Minor updates for IPA hardware layout; change servo twist for laser corrections to avoid collisions

File: ipa_demo_cell_description/urdf/ipa_ur_demo.urdf.xacro (robot description, xacro)
@@ -4,5 +4,5 @@
   <xacro:arg name="name" default="ipa_ur_demo"/>
   <!-- Endeffector name -->
-  <xacro:arg name="endeffector" default="welding_gun_lorch_scancontrol" />
+  <xacro:arg name="endeffector" default="welding_gun_lorch_scancontrol_3000" />
   <!-- <xacro:property name="endeffector" value="$(arg endeffector)" /> -->
   <!-- Robot model -->
@@ -86,5 +86,5 @@
   <xacro:property name="flange_welding_gun" value="${welding_gun_config['flange_welding_gun']}"/>
   <joint name="welding_gun_joint" type="fixed">
-    <parent link="wrist_3_link" />
+    <parent link="tcp_welding_gun_link" />
     <child link="welding_gun_link" />
     <origin xyz="${flange_welding_gun['x']}

File: ipa_moveit_config/srdf/ur_macro.srdf.xacro (robot description, xacro)
@@ -40,10 +40,10 @@
     </group_state>
     <group_state name="${prefix}pre_welding_configuration" group="${prefix}${name}_manipulator">
-      <joint name="${prefix}elbow_joint" value="1.744" />
-      <joint name="${prefix}shoulder_lift_joint" value="-1.506" />
-      <joint name="${prefix}shoulder_pan_joint" value="0.838" />
-      <joint name="${prefix}wrist_1_joint" value="-1.712" />
-      <joint name="${prefix}wrist_2_joint" value="-1.691" />
-      <joint name="${prefix}wrist_3_joint" value="-0.809" />
+      <joint name="${prefix}elbow_joint" value="2.22" />
+      <joint name="${prefix}shoulder_lift_joint" value="-1.93" />
+      <joint name="${prefix}shoulder_pan_joint" value="0.86" />
+      <joint name="${prefix}wrist_1_joint" value="-1.97" />
+      <joint name="${prefix}wrist_2_joint" value="-1.63" />
+      <joint name="${prefix}wrist_3_joint" value="0.72" />
     </group_state>
     <!--END EFFECTOR - Purpose - Represent information about an end effector.-->

Commit message: Switch to upstream ur xacro for initial positions support

File: ipa_demo_cell_description/urdf/ipa_ur_demo.urdf.xacro (robot description, xacro)
@@ -22,9 +22,9 @@
   <xacro:arg name="use_fake_hardware" default="false" />
   <xacro:arg name="fake_sensor_commands" default="false" />
+  <xacro:arg name="headless_mode" default="false" />
+  <xacro:arg name="initial_positions_file" default="$(find ipa_demo_cell_description)/config/$(arg robot_model)/ros2_control_initial_positions.yaml"/>
+  <xacro:property name="initial_positions_file" default="$(arg initial_positions_file)"/>
   <!-- Real robot hardware -->
-  <!-- TODO (christianlandgraf): Use ur_description as soon as PR#154 is merged -->
-  <!-- <xacro:include filename="$(find ur_description)/urdf/ur.urdf.xacro" /> -->
-  <!-- <xacro:include filename="$(find ur_description)/urdf/ur_macro.xacro" /> -->
-  <xacro:include filename="$(find ipa_demo_cell_description)/urdf/ur_macro.xacro" />
+  <xacro:include filename="$(find ur_description)/urdf/ur_macro.xacro" />
   <xacro:ur_robot
     prefix="$(arg prefix)"
@@ -39,5 +39,6 @@
     use_fake_hardware="$(arg use_fake_hardware)"
     fake_sensor_commands="$(arg fake_sensor_commands)"
-    initial_positions="${dict(shoulder_pan_joint=0.86, shoulder_lift_joint=-1.93, elbow_joint=2.22, wrist_1_joint=-1.97, wrist_2_joint=-1.63, wrist_3_joint=0.72)}"/>
+    headless_mode="$(arg headless_mode)"
+    initial_positions="${load_yaml(initial_positions_file)}" />
   <!-- Include the cell and attach it to the world-->
   <xacro:include filename="$(find ipa_demo_cell_description)/urdf/ipa_demo_env.urdf.xacro" />

Commit message: Updates for IPA hardware (#43)
* Update robot layout and calibration

* Add weld seam visualization

File: ipa_demo_cell_description/urdf/ipa_ur_demo.urdf.xacro (robot description, xacro)
@@ -44,11 +44,9 @@
   <xacro:include filename="$(find ipa_demo_cell_description)/urdf/ipa_demo_env.urdf.xacro" />
   <link name="world" />
-  <xacro:ipa_demo_env
-    prefix=""
-    use_fake_hardware="$(arg use_fake_hardware)" />
+  <xacro:ipa_demo_env prefix="" />
   <joint name="demo_env_joint" type="fixed">
     <parent link="world" />
     <child link="env_link" />
-    <origin xyz="0 0 0" rpy="${pi/2} 0 0"/>
+    <origin xyz="0 0 0" rpy="0 0 0"/>
   </joint>
   <!-- Attach UR to environment -->
@@ -56,5 +54,5 @@
     <parent link="env_link" />
     <child link="base_link" />
-    <origin xyz="-0.350 0.766 0" rpy="-${pi/2} -${pi/2} 0" />
+    <origin xyz="-0.350 0 0.813" rpy="0 0 ${-pi/2}" />
   </joint>
   <!-- Sensor calibration -->

Commit message: Update welding demo urdf xacro
Update `ur_robot` macro params

Remove "robot_platform_joint" as the updated `ur_robot` macro takes care
of connecting the robot to the provided parent link now.

Use `xacro.load_yaml` instead of deprecated `load_yaml` function

NOTE: these changes are required if the demo is run with an updated
version of the ur_description package that provides the `ur_robot` macro

File: ipa_demo_cell_description/urdf/ipa_ur_demo.urdf.xacro (robot description, xacro)
@@ -28,5 +28,7 @@
   <xacro:include filename="$(find ur_description)/urdf/ur_macro.xacro" />
   <xacro:ur_robot
-    prefix="$(arg prefix)"
+    name="$(arg name)"
+    tf_prefix="$(arg prefix)"
+    parent="env_link"
     joint_limits_parameters_file="$(arg joint_limit_params)"
     kinematics_parameters_file="$(arg kinematics_params)"
@@ -40,5 +42,7 @@
     fake_sensor_commands="$(arg fake_sensor_commands)"
     headless_mode="$(arg headless_mode)"
-    initial_positions="${load_yaml(initial_positions_file)}" />
+    initial_positions="${xacro.load_yaml(initial_positions_file)}">
+    <origin xyz="-0.350 0 0.813" rpy="0 0 ${-pi/2}" />
+  </xacro:ur_robot>
   <!-- Include the cell and attach it to the world-->
   <xacro:include filename="$(find ipa_demo_cell_description)/urdf/ipa_demo_env.urdf.xacro" />
@@ -50,13 +54,7 @@
     <origin xyz="0 0 0" rpy="0 0 0"/>
   </joint>
-  <!-- Attach UR to environment -->
-  <joint name="robot_platform_joint" type="fixed">
-    <parent link="env_link" />
-    <child link="base_link" />
-    <origin xyz="-0.350 0 0.813" rpy="0 0 ${-pi/2}" />
-  </joint>
   <!-- Sensor calibration -->
   <!-- Set the tcp according to Hand Eye Calibration-->
-  <xacro:property name="sensor_config" value="${load_yaml('$(arg calibration_config_file)')}" />
+  <xacro:property name="sensor_config" value="${xacro.load_yaml('$(arg calibration_config_file)')}" />
   <xacro:property name="tcp_sensor" value="${sensor_config['tcp_sensor']}"/>
   <link name="tcp_sensor_link" />
@@ -71,5 +69,5 @@
   </joint>
   <!-- Set the welding gun tool-->
-  <xacro:property name="welding_gun_config" value="${load_yaml('$(arg calibration_config_file)')}" />
+  <xacro:property name="welding_gun_config" value="${xacro.load_yaml('$(arg calibration_config_file)')}" />
   <xacro:property name="tcp_welding_gun" value="${welding_gun_config['tcp_welding_gun']}"/>
   <link name="tcp_welding_gun_link" />
